Commit message: Fix exo_model urdf

File: ros-ws/src/bringup_robot/urdf/exo_model.xacro.urdf (robot description, URDF)
Before this commit: robot exo_model, 2 links, 1 joints
Links:
- link base_link: mass None -> 5.0; geometry collision box size=0.2 ${base_bar_length} 0.2; visual box size=0.2 ${base_bar_length} 0.2

Commit message: Move inertia tag from base_link to dummy_link

File: ros-ws/src/bringup_robot/urdf/exo_model.xacro.urdf (robot description, URDF)
Before this commit: robot exo_model, 2 links, 1 joints
Links:
- link base_link: mass 5.0 -> None
- link dummy_link: mass None -> 5.0
